Commit message: 修改深度相机参数，取消近距离裁剪功能

File: car_2026/src/robot_description/urdf/robotcar_sensor_plugins.xacro (robot description, xacro)
@@ -51,5 +51,5 @@
   <xacro:property name="camera_update_rate" value="15.0"/>
   <xacro:property name="camera_hfov" value="1.0471975511965976"/>
-  <xacro:property name="camera_near" value="0.6"/>
+  <xacro:property name="camera_near" value="0.05"/>
   <xacro:property name="camera_far" value="8.0"/>
   <gazebo reference="base_link">

Commit message: 修改相机角度向上5度

File: car_2026/src/robot_description/urdf/robotcar_sensor_plugins.xacro (robot description, xacro)
@@ -55,5 +55,5 @@
   <gazebo reference="base_link">
     <sensor name="depth_camera_sensor" type="depth">
-      <pose>${camera_x} ${camera_y} ${camera_z} 0 0 0</pose>
+      <pose>${camera_x} ${camera_y} ${camera_z} 0 -0.0872665 0</pose>
       <always_on>true</always_on>
       <visualize>false</visualize>

File: car_2026/src/robot_description/urdf/robotcar_sensors.xacro (robot description, xacro)
@@ -41,5 +41,5 @@
     <parent link="base_link"/>
     <child link="camera_link"/>
-    <origin xyz="${camera_x} ${camera_y} ${camera_z}" rpy="0 0 0"/>
+    <origin xyz="${camera_x} ${camera_y} ${camera_z}" rpy="0 -0.0872665 0"/>
   </joint>
   <!-- REP-103 / ROS optical convention: +Z forward, +X right, +Y down. -->
